File: circuits/laser_controller.kicad_sch (KiCad schematic)
At the start: 0 parts

Commit message: chore(circuits): update laser controller release artifacts
Other:
- sheet LASER_BLUE ports: added MPD_RAW; removed none
- sheet LASER_GREEN ports: added MPD_RAW; removed none
- sheet LASER_IR ports: added MPD_RAW; removed none
- sheet LASER_RED ports: added MPD_RAW; removed none
- sheet POWER_IO ports: added MPD_RAW1, MPD_RAW2, MPD_RAW3, MPD_RAW4; removed none
- note added: "Global-label nets join the sheet pins (VOUT1..4, PWM1..4, ISENSE1..4, MPD_RAW1..4, MPD1..4, LASER_N1..4, CONVST, VBUS_5V). +5V / +3V3 / LASER_V+ / GND are global power. Each channel = 1 laser + current-sense + internal monitor PD + external/sample PD TIA."
- note removed: "Global-label nets join the sheet pins (VOUT1..4, PWM1..4, ISENSE1..4, MPD1..4, LASER_N1..4, CONVST, VBUS_5V). +5V / +3V3 / LASER_V+ / GND are global power. Each channel = 1 laser + current-sense + internal monitor PD + external/sample PD TIA."
- title: Laser Controller — 1ch x 4 wavelengths: on-board PD -> TIA + monitor-PD feedback + ESP32-S3 USB + 4x laser drivers -> Laser Controller
Changed lines of the file:
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@@
   (paper "A2")
   (title_block
-    (title "Laser Controller — 1ch x 4 wavelengths: on-board PD -> TIA + monitor-PD feedback + ESP32-S3 USB + 4x laser drivers")
+    (title "Laser Controller")
     (date "2026-06-24")
     (rev "v9")
@@
     (pin "LASER_N" output (at 302 78 0) (effects (font (size 1.0 1.0)) (justify left)))
     (pin "ISENSE" output (at 302 85 0) (effects (font (size 1.0 1.0)) (justify left)))
+    (pin "MPD_RAW" output (at 302 92 0) (effects (font (size 1.0 1.0)) (justify left)))
   )
   (sheet (at 240 124) (size 62 34) (stroke (width 0.254) (type solid)) (fill (color 0 0 0 0.0))
@@
     (pin "LASER_N" output (at 302 132 0) (effects (font (size 1.0 1.0)) (justify left)))
     (pin "ISENSE" output (at 302 139 0) (effects (font (size 1.0 1.0)) (justify left)))
+    (pin "MPD_RAW" output (at 302 146 0) (effects (font (size 1.0 1.0)) (justify left)))
   )
   (sheet (at 240 178) (size 62 34) (stroke (width 0.254) (type solid)) (fill (color 0 0 0 0.0))
@@
     (pin "LASER_N" output (at 302 186 0) (effects (font (size 1.0 1.0)) (justify left)))
     (pin "ISENSE" output (at 302 193 0) (effects (font (size 1.0 1.0)) (justify left)))
+    (pin "MPD_RAW" output (at 302 200 0) (effects (font (size 1.0 1.0)) (justify left)))
   )
   (sheet (at 240 232) (size 62 34) (stroke (width 0.254) (type solid)) (fill (color 0 0 0 0.0))
@@
     (pin "LASER_N" output (at 302 240 0) (effects (font (size 1.0 1.0)) (justify left)))
     (pin "ISENSE" output (at 302 247 0) (effects (font (size 1.0 1.0)) (justify left)))
+    (pin "MPD_RAW" output (at 302 254 0) (effects (font (size 1.0 1.0)) (justify left)))
   )
   (sheet (at 430 70) (size 95 118) (stroke (width 0.254) (type solid)) (fill (color 0 0 0 0.0))
@@
     (pin "VBUS_5V" output (at 430 169 180) (effects (font (size 1.0 1.0)) (justify right)))
   )
-  (sheet (at 430 256) (size 95 110) (stroke (width 0.254) (type solid)) (fill (color 0 0 0 0.0))
+  (sheet (at 430 256) (size 95 140) (stroke (width 0.254) (type solid)) (fill (color 0 0 0 0.0))
     (property "Sheetname" "POWER_IO" (at 430 253 0) (effects (font (size 1.4 1.4)) (justify left bottom)))
-    (property "Sheetfile" "power_io.kicad_sch" (at 430 370 0) (effects (font (size 1.0 1.0)) (justify left top)))
+    (property "Sheetfile" "power_io.kicad_sch" (at 430 400 0) (effects (font (size 1.0 1.0)) (justify left top)))
     (pin "VOUT1" input (at 430 264 180) (effects (font (size 1.0 1.0)) (justify right)))
     (pin "VOUT2" input (at 430 271 180) (effects (font (size 1.0 1.0)) (justify right)))
@@
     (pin "LASER_N3" input (at 430 320 180) (effects (font (size 1.0 1.0)) (justify right)))
     (pin "LASER_N4" input (at 430 327 180) (effects (font (size 1.0 1.0)) (justify right)))
-    (pin "MPD1" output (at 430 334 180) (effects (font (size 1.0 1.0)) (justify right)))
-    (pin "MPD2" output (at 430 341 180) (effects (font (size 1.0 1.0)) (justify right)))
-    (pin "MPD3" output (at 430 348 180) (effects (font (size 1.0 1.0)) (justify right)))
-    (pin "MPD4" output (at 430 355 180) (effects (font (size 1.0 1.0)) (justify right)))
+    (pin "MPD_RAW1" input (at 430 334 180) (effects (font (size 1.0 1.0)) (justify right)))
+    (pin "MPD_RAW2" input (at 430 341 180) (effects (font (size 1.0 1.0)) (justify right)))
+    (pin "MPD_RAW3" input (at 430 348 180) (effects (font (size 1.0 1.0)) (justify right)))
+    (pin "MPD_RAW4" input (at 430 355 180) (effects (font (size 1.0 1.0)) (justify right)))
+    (pin "MPD1" output (at 430 362 180) (effects (font (size 1.0 1.0)) (justify right)))
+    (pin "MPD2" output (at 430 369 180) (effects (font (size 1.0 1.0)) (justify right)))
+    (pin "MPD3" output (at 430 376 180) (effects (font (size 1.0 1.0)) (justify right)))
+    (pin "MPD4" output (at 430 383 180) (effects (font (size 1.0 1.0)) (justify right)))
   )
   (wire (pts (xy 122 78) (xy 130 78)) (stroke (width 0) (type default)))
@@
   (wire (pts (xy 302 85) (xy 310 85)) (stroke (width 0) (type default)))
   (global_label "ISENSE1" (shape bidirectional) (at 310 85 0) (effects (font (size 1.27 1.27)) (justify left)))
+  (wire (pts (xy 302 92) (xy 310 92)) (stroke (width 0) (type default)))
+  (global_label "MPD_RAW1" (shape bidirectional) (at 310 92 0) (effects (font (size 1.27 1.27)) (justify left)))
   (wire (pts (xy 240 132) (xy 232 132)) (stroke (width 0) (type default)))
   (global_label "PWM2" (shape bidirectional) (at 232 132 180) (effects (font (size 1.27 1.27)) (justify right)))
@@
   (wire (pts (xy 302 139) (xy 310 139)) (stroke (width 0) (type default)))
   (global_label "ISENSE2" (shape bidirectional) (at 310 139 0) (effects (font (size 1.27 1.27)) (justify left)))
+  (wire (pts (xy 302 146) (xy 310 146)) (stroke (width 0) (type default)))
+  (global_label "MPD_RAW2" (shape bidirectional) (at 310 146 0) (effects (font (size 1.27 1.27)) (justify left)))
   (wire (pts (xy 240 186) (xy 232 186)) (stroke (width 0) (type default)))
   (global_label "PWM3" (shape bidirectional) (at 232 186 180) (effects (font (size 1.27 1.27)) (justify right)))
@@
   (wire (pts (xy 302 193) (xy 310 193)) (stroke (width 0) (type default)))
   (global_label "ISENSE3" (shape bidirectional) (at 310 193 0) (effects (font (size 1.27 1.27)) (justify left)))
+  (wire (pts (xy 302 200) (xy 310 200)) (stroke (width 0) (type default)))
+  (global_label "MPD_RAW3" (shape bidirectional) (at 310 200 0) (effects (font (size 1.27 1.27)) (justify left)))
   (wire (pts (xy 240 240) (xy 232 240)) (stroke (width 0) (type default)))
   (global_label "PWM4" (shape bidirectional) (at 232 240 180) (effects (font (size 1.27 1.27)) (justify right)))
@@
   (wire (pts (xy 302 247) (xy 310 247)) (stroke (width 0) (type default)))
   (global_label "ISENSE4" (shape bidirectional) (at 310 247 0) (effects (font (size 1.27 1.27)) (justify left)))
+  (wire (pts (xy 302 254) (xy 310 254)) (stroke (width 0) (type default)))
+  (global_label "MPD_RAW4" (shape bidirectional) (at 310 254 0) (effects (font (size 1.27 1.27)) (justify left)))
   (wire (pts (xy 430 78) (xy 422 78)) (stroke (width 0) (type default)))
   (global_label "PWM1" (shape bidirectional) (at 422 78 180) (effects (font (size 1.27 1.27)) (justify right)))
@@
   (global_label "LASER_N4" (shape bidirectional) (at 422 327 180) (effects (font (size 1.27 1.27)) (justify right)))
   (wire (pts (xy 430 334) (xy 422 334)) (stroke (width 0) (type default)))
-  (global_label "MPD1" (shape bidirectional) (at 422 334 180) (effects (font (size 1.27 1.27)) (justify right)))
+  (global_label "MPD_RAW1" (shape bidirectional) (at 422 334 180) (effects (font (size 1.27 1.27)) (justify right)))
   (wire (pts (xy 430 341) (xy 422 341)) (stroke (width 0) (type default)))
-  (global_label "MPD2" (shape bidirectional) (at 422 341 180) (effects (font (size 1.27 1.27)) (justify right)))
+  (global_label "MPD_RAW2" (shape bidirectional) (at 422 341 180) (effects (font (size 1.27 1.27)) (justify right)))
   (wire (pts (xy 430 348) (xy 422 348)) (stroke (width 0) (type default)))
-  (global_label "MPD3" (shape bidirectional) (at 422 348 180) (effects (font (size 1.27 1.27)) (justify right)))
+  (global_label "MPD_RAW3" (shape bidirectional) (at 422 348 180) (effects (font (size 1.27 1.27)) (justify right)))
   (wire (pts (xy 430 355) (xy 422 355)) (stroke (width 0) (type default)))
-  (global_label "MPD4" (shape bidirectional) (at 422 355 180) (effects (font (size 1.27 1.27)) (justify right)))
+  (global_label "MPD_RAW4" (shape bidirectional) (at 422 355 180) (effects (font (size 1.27 1.27)) (justify right)))
+  (wire (pts (xy 430 362) (xy 422 362)) (stroke (width 0) (type default)))
+  (global_label "MPD1" (shape bidirectional) (at 422 362 180) (effects (font (size 1.27 1.27)) (justify right)))
+  (wire (pts (xy 430 369) (xy 422 369)) (stroke (width 0) (type default)))
+  (global_label "MPD2" (shape bidirectional) (at 422 369 180) (effects (font (size 1.27 1.27)) (justify right)))
+  (wire (pts (xy 430 376) (xy 422 376)) (stroke (width 0) (type default)))
+  (global_label "MPD3" (shape bidirectional) (at 422 376 180) (effects (font (size 1.27 1.27)) (justify right)))
+  (wire (pts (xy 430 383) (xy 422 383)) (stroke (width 0) (type default)))
+  (global_label "MPD4" (shape bidirectional) (at 422 383 180) (effects (font (size 1.27 1.27)) (justify right)))
   (text "LASER CONTROLLER  ·  Vivonics  ·  rev v9   —   1 channel x 4 wavelengths (IR / RED / GREEN / BLUE)  ·  TIA x4  ·  laser_driver x4  ·  monitor PD ADC x4  ·  mcu  ·  power_io" (at 40 30 0) (effects (font (size 2.4 2.4)) (justify left)))
-  (text "Global-label nets join the sheet pins (VOUT1..4, PWM1..4, ISENSE1..4, MPD1..4, LASER_N1..4, CONVST, VBUS_5V).   +5V / +3V3 / LASER_V+ / GND are global power.   Each channel = 1 laser + current-sense + internal monitor PD + external/sample PD TIA." (at 40 36 0) (effects (font (size 1.6 1.6)) (justify left)))
+  (text "Global-label nets join the sheet pins (VOUT1..4, PWM1..4, ISENSE1..4, MPD_RAW1..4, MPD1..4, LASER_N1..4, CONVST, VBUS_5V).   +5V / +3V3 / LASER_V+ / GND are global power.   Each channel = 1 laser + current-sense + internal monitor PD + external/sample PD TIA." (at 40 36 0) (effects (font (size 1.6 1.6)) (justify left)))
   (sheet_instances
     (path "/" (page "1"))

Commit message: fix(circuits): import mcu sheet and laser footprints
Other:
- sheet LASER_BLUE ports: added none; removed MPD_RAW
- sheet MCU_ESP32-S3 ports: added 3V3, 5V, IO10, IO11, IO12, IO15, IO16, IO2, IO3, IO4, IO5, IO6, IO7, IO8, IO9; removed CONVST, ISENSE1, ISENSE2, ISENSE3, ISENSE4, MPD1, MPD2, MPD3, MPD4, PWM1, PWM2, PWM3, PWM4, VBUS_5V
- note added: "Global-label nets join sheet pins (VOUT1..4, PWM1..4, ISENSE1..4, MPD_RAW1..3 plus open MPD_RAW4 header/front-end, MPD1..4, LASER_N1..4, CONVST, VBUS_5V, +3V3). MCU mapping: IO10/11/12/16=PWM1..4, IO4..7=ISENSE1..4, IO2/3/8/9=MPD1..4, IO15=CONVST."
- note added: "LASER CONTROLLER · Vivonics · rev v9 — 1 channel x 4 wavelengths (IR / RED / GREEN / BLUE) · TIA x4 · laser_driver x4 · monitor PD ADC x3+spare · mcu · power_io"
- note removed: "Global-label nets join the sheet pins (VOUT1..4, PWM1..4, ISENSE1..4, MPD_RAW1..4, MPD1..4, LASER_N1..4, CONVST, VBUS_5V). +5V / +3V3 / LASER_V+ / GND are global power. Each channel = 1 laser + current-sense + internal monitor PD + external/sample PD TIA."
- note removed: "LASER CONTROLLER · Vivonics · rev v9 — 1 channel x 4 wavelengths (IR / RED / GREEN / BLUE) · TIA x4 · laser_driver x4 · monitor PD ADC x4 · mcu · power_io"

Commit message: save laser controller schematic and layout state
Other:
- sheet MCU_ESP32-S3 ports: added IO17, IO18, IO21, IO38, IO47, IO48; removed none
- sheet POWER_IO ports: added ADC_BUSY, ADC_CS, ADC_MISO_A, ADC_MISO_B, ADC_RESET, ADC_SCLK; removed none
- note added: "Global-label nets join sheet pins (VOUT1..4, ADC_SCLK/CS/MISO_A/MISO_B/BUSY/RESET, PWM1..4, ISENSE1..4, MPD_RAW1..3 plus open MPD_RAW4, MPD1..4, LASER_N1..4, CONVST, VBUS_5V, +3V3)."
- note added: "LASER CONTROLLER · Vivonics · rev v9 — 1 channel x 4 wavelengths (IR / RED / GREEN / BLUE) · TIA x4 · laser_driver x4 · AD7606-4 signal ADC · monitor PD ADC x3+spare · mcu · power_io"
- note removed: "Global-label nets join sheet pins (VOUT1..4, PWM1..4, ISENSE1..4, MPD_RAW1..3 plus open MPD_RAW4 header/front-end, MPD1..4, LASER_N1..4, CONVST, VBUS_5V, +3V3). MCU mapping: IO10/11/12/16=PWM1..4, IO4..7=ISENSE1..4, IO2/3/8/9=MPD1..4, IO15=CONVST."
- note removed: "LASER CONTROLLER · Vivonics · rev v9 — 1 channel x 4 wavelengths (IR / RED / GREEN / BLUE) · TIA x4 · laser_driver x4 · monitor PD ADC x3+spare · mcu · power_io"
Changed lines of the file:
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@@
     (pin "5V" output (at 430.53 176.53 180) (effects (font (size 1.0 1.0)) (justify right)))
     (pin "3V3" input (at 430.53 184.15 180) (effects (font (size 1.0 1.0)) (justify right)))
+    (pin "IO17" output (at 525.78 77.47 0) (effects (font (size 1.0 1.0)) (justify left)))
+    (pin "IO18" output (at 525.78 85.09 0) (effects (font (size 1.0 1.0)) (justify left)))
+    (pin "IO21" input (at 525.78 92.71 0) (effects (font (size 1.0 1.0)) (justify left)))
+    (pin "IO38" input (at 525.78 100.33 0) (effects (font (size 1.0 1.0)) (justify left)))
+    (pin "IO47" input (at 525.78 107.95 0) (effects (font (size 1.0 1.0)) (justify left)))
+    (pin "IO48" output (at 525.78 115.57 0) (effects (font (size 1.0 1.0)) (justify left)))
   )
   (sheet (at 430.53 219.71) (size 95.25 139.7) (stroke (width 0.254) (type solid)) (fill (color 0 0 0 0.0))
@@
     (pin "MPD3" output (at 430.53 328.93 180) (effects (font (size 1.0 1.0)) (justify right)))
     (pin "MPD4" output (at 430.53 335.28 180) (effects (font (size 1.0 1.0)) (justify right)))
+    (pin "ADC_SCLK" input (at 525.78 227.33 0) (effects (font (size 1.0 1.0)) (justify left)))
+    (pin "ADC_CS" input (at 525.78 233.68 0) (effects (font (size 1.0 1.0)) (justify left)))
+    (pin "ADC_MISO_A" output (at 525.78 240.03 0) (effects (font (size 1.0 1.0)) (justify left)))
+    (pin "ADC_MISO_B" output (at 525.78 246.38 0) (effects (font (size 1.0 1.0)) (justify left)))
+    (pin "ADC_BUSY" output (at 525.78 252.73 0) (effects (font (size 1.0 1.0)) (justify left)))
+    (pin "ADC_RESET" input (at 525.78 259.08 0) (effects (font (size 1.0 1.0)) (justify left)))
   )
   (wire (pts (xy 121.92 77.47) (xy 129.54 77.47)) (stroke (width 0) (type default)))
@@
   (wire (pts (xy 430.53 184.15) (xy 422.91 184.15)) (stroke (width 0) (type default)))
   (global_label "+3V3" (shape bidirectional) (at 422.91 184.15 180) (effects (font (size 1.27 1.27)) (justify right)))
+  (wire (pts (xy 525.78 77.47) (xy 533.4 77.47)) (stroke (width 0) (type default)))
+  (global_label "ADC_SCLK" (shape bidirectional) (at 533.4 77.47 0) (effects (font (size 1.27 1.27)) (justify left)))
+  (wire (pts (xy 525.78 85.09) (xy 533.4 85.09)) (stroke (width 0) (type default)))
+  (global_label "ADC_CS" (shape bidirectional) (at 533.4 85.09 0) (effects (font (size 1.27 1.27)) (justify left)))
+  (wire (pts (xy 525.78 92.71) (xy 533.4 92.71)) (stroke (width 0) (type default)))
+  (global_label "ADC_MISO_A" (shape bidirectional) (at 533.4 92.71 0) (effects (font (size 1.27 1.27)) (justify left)))
+  (wire (pts (xy 525.78 100.33) (xy 533.4 100.33)) (stroke (width 0) (type default)))
+  (global_label "ADC_MISO_B" (shape bidirectional) (at 533.4 100.33 0) (effects (font (size 1.27 1.27)) (justify left)))
+  (wire (pts (xy 525.78 107.95) (xy 533.4 107.95)) (stroke (width 0) (type default)))
+  (global_label "ADC_BUSY" (shape bidirectional) (at 533.4 107.95 0) (effects (font (size 1.27 1.27)) (justify left)))
+  (wire (pts (xy 525.78 115.57) (xy 533.4 115.57)) (stroke (width 0) (type default)))
+  (global_label "ADC_RESET" (shape bidirectional) (at 533.4 115.57 0) (effects (font (size 1.27 1.27)) (justify left)))
   (wire (pts (xy 430.53 227.33) (xy 422.91 227.33)) (stroke (width 0) (type default)))
   (global_label "VOUT1" (shape bidirectional) (at 422.91 227.33 180) (effects (font (size 1.27 1.27)) (justify right)))
@@
   (wire (pts (xy 430.53 335.28) (xy 422.91 335.28)) (stroke (width 0) (type default)))
   (global_label "MPD4" (shape bidirectional) (at 422.91 335.28 180) (effects (font (size 1.27 1.27)) (justify right)))
-  (text "LASER CONTROLLER  ·  Vivonics  ·  rev v9   —   1 channel x 4 wavelengths (IR / RED / GREEN / BLUE)  ·  TIA x4  ·  laser_driver x4  ·  monitor PD ADC x3+spare  ·  mcu  ·  power_io" (at 40 30 0) (effects (font (size 2.4 2.4)) (justify left)))
-  (text "Global-label nets join sheet pins (VOUT1..4, PWM1..4, ISENSE1..4, MPD_RAW1..3 plus open MPD_RAW4 header/front-end, MPD1..4, LASER_N1..4, CONVST, VBUS_5V, +3V3). MCU mapping: IO10/11/12/16=PWM1..4, IO4..7=ISENSE1..4, IO2/3/8/9=MPD1..4, IO15=CONVST." (at 40 36 0) (effects (font (size 1.6 1.6)) (justify left)))
+  (wire (pts (xy 525.78 227.33) (xy 533.4 227.33)) (stroke (width 0) (type default)))
+  (global_label "ADC_SCLK" (shape bidirectional) (at 533.4 227.33 0) (effects (font (size 1.27 1.27)) (justify left)))
+  (wire (pts (xy 525.78 233.68) (xy 533.4 233.68)) (stroke (width 0) (type default)))
+  (global_label "ADC_CS" (shape bidirectional) (at 533.4 233.68 0) (effects (font (size 1.27 1.27)) (justify left)))
+  (wire (pts (xy 525.78 240.03) (xy 533.4 240.03)) (stroke (width 0) (type default)))
+  (global_label "ADC_MISO_A" (shape bidirectional) (at 533.4 240.03 0) (effects (font (size 1.27 1.27)) (justify left)))
+  (wire (pts (xy 525.78 246.38) (xy 533.4 246.38)) (stroke (width 0) (type default)))
+  (global_label "ADC_MISO_B" (shape bidirectional) (at 533.4 246.38 0) (effects (font (size 1.27 1.27)) (justify left)))
+  (wire (pts (xy 525.78 252.73) (xy 533.4 252.73)) (stroke (width 0) (type default)))
+  (global_label "ADC_BUSY" (shape bidirectional) (at 533.4 252.73 0) (effects (font (size 1.27 1.27)) (justify left)))
+  (wire (pts (xy 525.78 259.08) (xy 533.4 259.08)) (stroke (width 0) (type default)))
+  (global_label "ADC_RESET" (shape bidirectional) (at 533.4 259.08 0) (effects (font (size 1.27 1.27)) (justify left)))
+  (text "LASER CONTROLLER  ·  Vivonics  ·  rev v9   —   1 channel x 4 wavelengths (IR / RED / GREEN / BLUE)  ·  TIA x4  ·  laser_driver x4  ·  AD7606-4 signal ADC  ·  monitor PD ADC x3+spare  ·  mcu  ·  power_io" (at 40 30 0) (effects (font (size 2.4 2.4)) (justify left)))
+  (text "Global-label nets join sheet pins (VOUT1..4, ADC_SCLK/CS/MISO_A/MISO_B/BUSY/RESET, PWM1..4, ISENSE1..4, MPD_RAW1..3 plus open MPD_RAW4, MPD1..4, LASER_N1..4, CONVST, VBUS_5V, +3V3)." (at 40 36 0) (effects (font (size 1.6 1.6)) (justify left)))
   (sheet_instances
     (path "/" (page "1"))
