File: circuits/laser_controller.kicad_sch (KiCad schematic)
At the start: 0 parts

Commit message: save current laser controller recovery state
Other:
- sheet POWER_IO ports: added none; removed LASER_N1, LASER_N2, LASER_N3, LASER_N4
- note added: "Global-label nets join sheet pins (VOUT1..4, ADC_SCLK/CS/MISO_A/MISO_B/BUSY/RESET, PWM1..4, ISENSE1..4, MPD_RAW1..3 plus spare MPD_RAW4, MPD1..4, LASER_N1..4, CONVST, VBUS_5V, +3V3)."
- note removed: "Global-label nets join sheet pins (VOUT1..4, ADC_SCLK/CS/MISO_A/MISO_B/BUSY/RESET, PWM1..4, ISENSE1..4, MPD_RAW1..3 plus open MPD_RAW4, MPD1..4, LASER_N1..4, CONVST, VBUS_5V, +3V3)."
Changed lines of the file:
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@@
     (pin "CONVST" input (at 430.53 252.73 180) (effects (font (size 1.0 1.0)) (justify right)))
     (pin "VBUS_5V" input (at 430.53 259.08 180) (effects (font (size 1.0 1.0)) (justify right)))
-    (pin "LASER_N1" input (at 430.53 265.43 180) (effects (font (size 1.0 1.0)) (justify right)))
-    (pin "LASER_N2" input (at 430.53 271.78 180) (effects (font (size 1.0 1.0)) (justify right)))
-    (pin "LASER_N3" input (at 430.53 278.13 180) (effects (font (size 1.0 1.0)) (justify right)))
-    (pin "LASER_N4" input (at 430.53 284.48 180) (effects (font (size 1.0 1.0)) (justify right)))
-    (pin "MPD_RAW1" input (at 430.53 290.83 180) (effects (font (size 1.0 1.0)) (justify right)))
-    (pin "MPD_RAW2" input (at 430.53 297.18 180) (effects (font (size 1.0 1.0)) (justify right)))
-    (pin "MPD_RAW3" input (at 430.53 303.53 180) (effects (font (size 1.0 1.0)) (justify right)))
-    (pin "MPD_RAW4" input (at 430.53 309.88 180) (effects (font (size 1.0 1.0)) (justify right)))
-    (pin "MPD1" output (at 430.53 316.23 180) (effects (font (size 1.0 1.0)) (justify right)))
-    (pin "MPD2" output (at 430.53 322.58 180) (effects (font (size 1.0 1.0)) (justify right)))
-    (pin "MPD3" output (at 430.53 328.93 180) (effects (font (size 1.0 1.0)) (justify right)))
-    (pin "MPD4" output (at 430.53 335.28 180) (effects (font (size 1.0 1.0)) (justify right)))
+    (pin "MPD_RAW1" input (at 430.53 265.43 180) (effects (font (size 1.0 1.0)) (justify right)))
+    (pin "MPD_RAW2" input (at 430.53 271.78 180) (effects (font (size 1.0 1.0)) (justify right)))
+    (pin "MPD_RAW3" input (at 430.53 278.13 180) (effects (font (size 1.0 1.0)) (justify right)))
+    (pin "MPD_RAW4" input (at 430.53 284.48 180) (effects (font (size 1.0 1.0)) (justify right)))
+    (pin "MPD1" output (at 430.53 290.83 180) (effects (font (size 1.0 1.0)) (justify right)))
+    (pin "MPD2" output (at 430.53 297.18 180) (effects (font (size 1.0 1.0)) (justify right)))
+    (pin "MPD3" output (at 430.53 303.53 180) (effects (font (size 1.0 1.0)) (justify right)))
+    (pin "MPD4" output (at 430.53 309.88 180) (effects (font (size 1.0 1.0)) (justify right)))
     (pin "ADC_SCLK" input (at 525.78 227.33 0) (effects (font (size 1.0 1.0)) (justify left)))
     (pin "ADC_CS" input (at 525.78 233.68 0) (effects (font (size 1.0 1.0)) (justify left)))
@@
   (global_label "VBUS_5V" (shape bidirectional) (at 422.91 259.08 180) (effects (font (size 1.27 1.27)) (justify right)))
   (wire (pts (xy 430.53 265.43) (xy 422.91 265.43)) (stroke (width 0) (type default)))
-  (global_label "LASER_N1" (shape bidirectional) (at 422.91 265.43 180) (effects (font (size 1.27 1.27)) (justify right)))
+  (global_label "MPD_RAW1" (shape bidirectional) (at 422.91 265.43 180) (effects (font (size 1.27 1.27)) (justify right)))
   (wire (pts (xy 430.53 271.78) (xy 422.91 271.78)) (stroke (width 0) (type default)))
-  (global_label "LASER_N2" (shape bidirectional) (at 422.91 271.78 180) (effects (font (size 1.27 1.27)) (justify right)))
+  (global_label "MPD_RAW2" (shape bidirectional) (at 422.91 271.78 180) (effects (font (size 1.27 1.27)) (justify right)))
   (wire (pts (xy 430.53 278.13) (xy 422.91 278.13)) (stroke (width 0) (type default)))
-  (global_label "LASER_N3" (shape bidirectional) (at 422.91 278.13 180) (effects (font (size 1.27 1.27)) (justify right)))
+  (global_label "MPD_RAW3" (shape bidirectional) (at 422.91 278.13 180) (effects (font (size 1.27 1.27)) (justify right)))
   (wire (pts (xy 430.53 284.48) (xy 422.91 284.48)) (stroke (width 0) (type default)))
-  (global_label "LASER_N4" (shape bidirectional) (at 422.91 284.48 180) (effects (font (size 1.27 1.27)) (justify right)))
+  (global_label "MPD_RAW4" (shape bidirectional) (at 422.91 284.48 180) (effects (font (size 1.27 1.27)) (justify right)))
   (wire (pts (xy 430.53 290.83) (xy 422.91 290.83)) (stroke (width 0) (type default)))
-  (global_label "MPD_RAW1" (shape bidirectional) (at 422.91 290.83 180) (effects (font (size 1.27 1.27)) (justify right)))
+  (global_label "MPD1" (shape bidirectional) (at 422.91 290.83 180) (effects (font (size 1.27 1.27)) (justify right)))
   (wire (pts (xy 430.53 297.18) (xy 422.91 297.18)) (stroke (width 0) (type default)))
-  (global_label "MPD_RAW2" (shape bidirectional) (at 422.91 297.18 180) (effects (font (size 1.27 1.27)) (justify right)))
+  (global_label "MPD2" (shape bidirectional) (at 422.91 297.18 180) (effects (font (size 1.27 1.27)) (justify right)))
   (wire (pts (xy 430.53 303.53) (xy 422.91 303.53)) (stroke (width 0) (type default)))
-  (global_label "MPD_RAW3" (shape bidirectional) (at 422.91 303.53 180) (effects (font (size 1.27 1.27)) (justify right)))
+  (global_label "MPD3" (shape bidirectional) (at 422.91 303.53 180) (effects (font (size 1.27 1.27)) (justify right)))
   (wire (pts (xy 430.53 309.88) (xy 422.91 309.88)) (stroke (width 0) (type default)))
-  (global_label "MPD_RAW4" (shape bidirectional) (at 422.91 309.88 180) (effects (font (size 1.27 1.27)) (justify right)))
-  (wire (pts (xy 430.53 316.23) (xy 422.91 316.23)) (stroke (width 0) (type default)))
-  (global_label "MPD1" (shape bidirectional) (at 422.91 316.23 180) (effects (font (size 1.27 1.27)) (justify right)))
-  (wire (pts (xy 430.53 322.58) (xy 422.91 322.58)) (stroke (width 0) (type default)))
-  (global_label "MPD2" (shape bidirectional) (at 422.91 322.58 180) (effects (font (size 1.27 1.27)) (justify right)))
-  (wire (pts (xy 430.53 328.93) (xy 422.91 328.93)) (stroke (width 0) (type default)))
-  (global_label "MPD3" (shape bidirectional) (at 422.91 328.93 180) (effects (font (size 1.27 1.27)) (justify right)))
-  (wire (pts (xy 430.53 335.28) (xy 422.91 335.28)) (stroke (width 0) (type default)))
-  (global_label "MPD4" (shape bidirectional) (at 422.91 335.28 180) (effects (font (size 1.27 1.27)) (justify right)))
+  (global_label "MPD4" (shape bidirectional) (at 422.91 309.88 180) (effects (font (size 1.27 1.27)) (justify right)))
   (wire (pts (xy 525.78 227.33) (xy 533.4 227.33)) (stroke (width 0) (type default)))
   (global_label "ADC_SCLK" (shape bidirectional) (at 533.4 227.33 0) (effects (font (size 1.27 1.27)) (justify left)))
@@
   (global_label "ADC_RESET" (shape bidirectional) (at 533.4 259.08 0) (effects (font (size 1.27 1.27)) (justify left)))
   (text "LASER CONTROLLER  ·  Vivonics  ·  rev v9   —   1 channel x 4 wavelengths (IR / RED / GREEN / BLUE)  ·  TIA x4  ·  laser_driver x4  ·  AD7606-4 signal ADC  ·  monitor PD ADC x3+spare  ·  mcu  ·  power_io" (at 40 30 0) (effects (font (size 2.4 2.4)) (justify left)))
-  (text "Global-label nets join sheet pins (VOUT1..4, ADC_SCLK/CS/MISO_A/MISO_B/BUSY/RESET, PWM1..4, ISENSE1..4, MPD_RAW1..3 plus open MPD_RAW4, MPD1..4, LASER_N1..4, CONVST, VBUS_5V, +3V3)." (at 40 36 0) (effects (font (size 1.6 1.6)) (justify left)))
+  (text "Global-label nets join sheet pins (VOUT1..4, ADC_SCLK/CS/MISO_A/MISO_B/BUSY/RESET, PWM1..4, ISENSE1..4, MPD_RAW1..3 plus spare MPD_RAW4, MPD1..4, LASER_N1..4, CONVST, VBUS_5V, +3V3)." (at 40 36 0) (effects (font (size 1.6 1.6)) (justify left)))
   (sheet_instances
     (path "/" (page "1"))
