File: circuits/laser_controller.kicad_sch (KiCad schematic)
At the start: 0 parts

Commit message: Checkpoint laser controller fab parity package
Parts:
- added H1, H2: M3, MountingHole:MountingHole_3.2mm_M3, symbol viv:MOUNTING_HOLE_PAD
Connections:
- new net GND: H1.1, H2.1
Changed lines of the file:
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@@
     (pin "ADC_RESET" input (at 525.78 259.08 0) (effects (font (size 1.0 1.0)) (justify left)))
+  )
+  (symbol (lib_id "viv:MOUNTING_HOLE_PAD") (at 552.45 382.27 0) (unit 1)
+    (in_bom yes) (on_board yes) (dnp no)
+    (property "Reference" "H1" (at 549.25 377.07 0) (effects (font (size 1.0 1.0)) (justify left)))
+    (property "Value" "M3" (at 549.25 386.67 0) (effects (font (size 1.0 1.0)) (justify left)))
+    (property "Footprint" "MountingHole:MountingHole_3.2mm_M3" (at 552.45 382.27 0) (effects (font (size 1.0 1.0)) hide))
+    (property "Datasheet" "" (at 552.45 382.27 0) (effects (font (size 1.0 1.0)) hide))
+    (property "Part Number" "" (at 552.45 382.27 0) (effects (font (size 1.0 1.0)) hide))
+    (property "LCSC" "" (at 552.45 382.27 0) (effects (font (size 1.0 1.0)) hide))
+    (pin "1")
+    (instances
+      (project "laser_controller"
+        (path "/c1d2e3f4-6000-4000-a000-000000000001" (reference "H1") (unit 1))
+      )
+    )
+  )
+  (wire (pts (xy 552.45 382.27) (xy 552.45 388.62)) (stroke (width 0) (type default)))
+  (symbol (lib_id "viv:GND") (at 552.45 388.62 0) (unit 1)
+    (in_bom no) (on_board yes) (dnp no)
+    (property "Reference" "#PWR0339" (at 552.45 391.62 0) (effects (font (size 1.0 1.0)) hide))
+    (property "Value" "GND" (at 552.45 392.82 0) (effects (font (size 1.27 1.27))))
+    (property "Footprint" "" (at 0 0 0) (effects (font (size 1.0 1.0)) hide))
+    (property "Datasheet" "" (at 0 0 0) (effects (font (size 1.0 1.0)) hide))
+    (pin "1")
+    (instances
+      (project "laser_controller"
+        (path "/c1d2e3f4-6000-4000-a000-000000000001" (reference "#PWR0339") (unit 1))
+      )
+    )
+  )
+  (symbol (lib_id "viv:MOUNTING_HOLE_PAD") (at 571.5 382.27 0) (unit 1)
+    (in_bom yes) (on_board yes) (dnp no)
+    (property "Reference" "H2" (at 568.3 377.07 0) (effects (font (size 1.0 1.0)) (justify left)))
+    (property "Value" "M3" (at 568.3 386.67 0) (effects (font (size 1.0 1.0)) (justify left)))
+    (property "Footprint" "MountingHole:MountingHole_3.2mm_M3" (at 571.5 382.27 0) (effects (font (size 1.0 1.0)) hide))
+    (property "Datasheet" "" (at 571.5 382.27 0) (effects (font (size 1.0 1.0)) hide))
+    (property "Part Number" "" (at 571.5 382.27 0) (effects (font (size 1.0 1.0)) hide))
+    (property "LCSC" "" (at 571.5 382.27 0) (effects (font (size 1.0 1.0)) hide))
+    (pin "1")
+    (instances
+      (project "laser_controller"
+        (path "/c1d2e3f4-6000-4000-a000-000000000001" (reference "H2") (unit 1))
+      )
+    )
+  )
+  (wire (pts (xy 571.5 382.27) (xy 571.5 388.62)) (stroke (width 0) (type default)))
+  (symbol (lib_id "viv:GND") (at 571.5 388.62 0) (unit 1)
+    (in_bom no) (on_board yes) (dnp no)
+    (property "Reference" "#PWR0340" (at 571.5 391.62 0) (effects (font (size 1.0 1.0)) hide))
+    (property "Value" "GND" (at 571.5 392.82 0) (effects (font (size 1.27 1.27))))
+    (property "Footprint" "" (at 0 0 0) (effects (font (size 1.0 1.0)) hide))
+    (property "Datasheet" "" (at 0 0 0) (effects (font (size 1.0 1.0)) hide))
+    (pin "1")
+    (instances
+      (project "laser_controller"
+        (path "/c1d2e3f4-6000-4000-a000-000000000001" (reference "#PWR0340") (unit 1))
+      )
+    )
   )
   (wire (pts (xy 121.92 77.47) (xy 129.54 77.47)) (stroke (width 0) (type default)))
