File: circuits/laser_green.kicad_sch (KiCad schematic)
At the start: 11 parts, among them Q3 AO3400A, U7 TLV9001

Commit message: Limit laser command current per channel
Parts:
- R31: value 30k LIMIT -> 3k LIMIT; LCSC C22984 -> C4211; Part Number 0603WAF3002T5E -> 0603WAF3001T5E
Other:
- note added: "PWM_IN → R21/C21 with R22 3k LIMIT → +IN (full-scale ≈0.76V, ≈76mA) ; −IN = FB (sense top)."
- note removed: "PWM_IN → R21/C21 with R22 30k limiter → +IN (full-scale ≈2.48V, ≈248mA) ; −IN = FB (sense top)."
Changed lines of the file:
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@@
     (in_bom yes) (on_board yes) (dnp no)
     (property "Reference" "R31" (at 203.72 157.35 0) (effects (font (size 1.0 1.0)) (justify left)))
-    (property "Value" "30k LIMIT" (at 203.72 160.15 0) (effects (font (size 1.0 1.0)) (justify left)))
+    (property "Value" "3k LIMIT" (at 203.72 160.15 0) (effects (font (size 1.0 1.0)) (justify left)))
     (property "Footprint" "Resistor_SMD:R_0603_1608Metric_Pad0.98x0.95mm_HandSolder" (at 198.12 158.75 0) (effects (font (size 1.0 1.0)) hide))
     (property "Datasheet" "" (at 198.12 158.75 0) (effects (font (size 1.0 1.0)) hide))
-    (property "Part Number" "0603WAF3002T5E" (at 198.12 158.75 0) (effects (font (size 1.0 1.0)) hide))
-    (property "LCSC" "C22984" (at 198.12 158.75 0) (effects (font (size 1.0 1.0)) hide))
+    (property "Part Number" "0603WAF3001T5E" (at 198.12 158.75 0) (effects (font (size 1.0 1.0)) hide))
+    (property "LCSC" "C4211" (at 198.12 158.75 0) (effects (font (size 1.0 1.0)) hide))
     (pin "1")
     (pin "2")
@@
   (label "LOUT" (at 222.25 180.34 0) (effects (font (size 1.27 1.27)) (justify left bottom)))
   (text "Laser Driver  —  TLV9001 + AO3400A constant-current sink  ·  I = V_ctrl / 10Ω  ·  reused 4× (IR / RED / GREEN / BLUE)" (at 150 114 0) (effects (font (size 2.0 2.0)) (justify left)))
-  (text "PWM_IN → R21/C21 with R22 30k limiter → +IN (full-scale ≈2.48V, ≈248mA) ;  −IN = FB (sense top)." (at 150 120 0) (effects (font (size 1.3 1.3)) (justify left)))
+  (text "PWM_IN → R21/C21 with R22 3k LIMIT → +IN (full-scale ≈0.76V, ≈76mA) ;  −IN = FB (sense top)." (at 150 120 0) (effects (font (size 1.3 1.3)) (justify left)))
   (text "TLV9001 out → R31 → Q1 gate ; source → 10Ω 2W sense → GND.  CC = loop comp (FB↔LOUT, tune in bring-up)." (at 150 125 0) (effects (font (size 1.3 1.3)) (justify left)))
   (text "Direct TO-can footprint is the board-mounted laser source connection; no separate laser/MPD harness header is populated." (at 150 130 0) (effects (font (size 1.3 1.3)) (justify left)))

Commit message: Checkpoint laser controller fab parity package
Parts:
- removed LD3: PLT5 520EB_P TO56 LASER+MPD, OptoDevice:LaserDiode_TO56-3, symbol viv:LASER_CAN_MON_PD
- added R29: 1k, Resistor_SMD:R_0603_1608Metric_Pad0.98x0.95mm_HandSolder, symbol viv:R_H
- LD3: renamed from R29; value 1k -> PLT5 520EB_P TO56 LASER+MPD; footprint Resistor_SMD:R_0603_1608Metric_Pad0.98x0.95mm_HandSolder -> OptoDevice:LaserDiode_TO56-3; symbol viv:R_H -> viv:LASER_CAN_MON_PD; LCSC C2907002 -> (none); Part Number FRC0603F1001TS -> PLT5 520EB_P; now left out of the parts list
Connections:
- net FB: now also R29.1; no longer LD3.1
- net ISENSE: now also R29.2; no longer LD3.2
- net LASER_N: now also LD3.1 (LD_K)
- net LASER_V+: now also LD3.2 (LD_A/PD_K/CASE)
- net MPD_RAW: now also LD3.3 (PD_A)
- net CMD_FILTER: now reaches C24.1, R30.2, R31.1, U7.3 (+)
- net GATE: now reaches Q3.1 (G), R27.2
Changed lines of the file:
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@@
   (junction (at 193.04 146.05) (diameter 0) (color 0 0 0 0))
   (junction (at 222.25 152.4) (diameter 0) (color 0 0 0 0))
+  (label "CMD_FILTER" (at 187.96 154.94 0) (effects (font (size 1.27 1.27)) (justify left bottom)))
+  (label "LOUT" (at 228.6 152.4 0) (effects (font (size 1.27 1.27)) (justify left bottom)))
+  (label "GATE" (at 248.92 152.4 0) (effects (font (size 1.27 1.27)) (justify left bottom)))
   (hierarchical_label "PWM_IN" (shape input) (at 162.56 154.94 0) (effects (font (size 1.27 1.27)) (justify right)))
   (hierarchical_label "ISENSE" (shape output) (at 283.21 165.1 0) (effects (font (size 1.27 1.27)) (justify left)))

Commit message: Checkpoint schematic warning hygiene
Parts:
- removed U7: TLV9001, Package_TO_SOT_SMD:SOT-23-5, symbol viv:TLV9001_SOT23_5
- added R29: 1k, Resistor_SMD:R_0603_1608Metric_Pad0.98x0.95mm_HandSolder, symbol viv:R_H
- U7: renamed from R29; value 1k -> TLV9001; footprint Resistor_SMD:R_0603_1608Metric_Pad0.98x0.95mm_HandSolder -> Package_TO_SOT_SMD:SOT-23-5; symbol viv:R_H -> viv:TLV9001_SOT23_5; LCSC C2907002 -> C398363; Part Number FRC0603F1001TS -> TLV9001IDBVR
Connections:
- net +5V: now also U7.5 (V+)
- net CMD_FILTER: now also U7.3 (+)
- net FB: now also U7.4 (-), R29.1; no longer U7.1
- net GND: now also U7.2 (V-)
- net ISENSE: now also R29.2; no longer U7.2
- net LOUT: now also U7.1
Changed lines of the file:
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@@
   (wire (pts (xy 187.96 167.64) (xy 187.96 172.72)) (stroke (width 0) (type default)))
   (wire (pts (xy 198.12 162.56) (xy 198.12 167.64)) (stroke (width 0) (type default)))
-  (wire (pts (xy 217.17 152.4) (xy 228.6 152.4)) (stroke (width 0) (type default)))
-  (wire (pts (xy 236.22 152.4) (xy 248.92 152.4)) (stroke (width 0) (type default)))
+  (wire (pts (xy 217.17 152.4) (xy 223.52 152.4)) (stroke (width 0) (type default)))
+  (wire (pts (xy 223.52 152.4) (xy 228.6 152.4)) (stroke (width 0) (type default)))
+  (wire (pts (xy 236.22 152.4) (xy 242.57 152.4)) (stroke (width 0) (type default)))
+  (wire (pts (xy 242.57 152.4) (xy 248.92 152.4)) (stroke (width 0) (type default)))
   (wire (pts (xy 254 157.48) (xy 254 163.83)) (stroke (width 0) (type default)))
   (wire (pts (xy 254 171.45) (xy 254 176.53)) (stroke (width 0) (type default)))
   (wire (pts (xy 254 163.83) (xy 270.51 163.83)) (stroke (width 0) (type default)))
   (wire (pts (xy 270.51 163.83) (xy 270.51 165.1)) (stroke (width 0) (type default)))
+  (wire (pts (xy 223.52 152.4) (xy 223.52 144.78)) (stroke (width 0) (type default)))
+  (wire (pts (xy 242.57 152.4) (xy 242.57 144.78)) (stroke (width 0) (type default)))
   (wire (pts (xy 167.64 154.94) (xy 162.56 154.94)) (stroke (width 0) (type default)))
   (wire (pts (xy 278.13 165.1) (xy 283.21 165.1)) (stroke (width 0) (type default)))
@@
   (junction (at 254 163.83) (diameter 0) (color 0 0 0 0))
   (junction (at 217.17 152.4) (diameter 0) (color 0 0 0 0))
+  (junction (at 223.52 152.4) (diameter 0) (color 0 0 0 0))
+  (junction (at 242.57 152.4) (diameter 0) (color 0 0 0 0))
   (junction (at 193.04 146.05) (diameter 0) (color 0 0 0 0))
   (junction (at 222.25 152.4) (diameter 0) (color 0 0 0 0))
   (label "CMD_FILTER" (at 187.96 154.94 0) (effects (font (size 1.27 1.27)) (justify left bottom)))
-  (label "LOUT" (at 228.6 152.4 0) (effects (font (size 1.27 1.27)) (justify left bottom)))
-  (label "GATE" (at 248.92 152.4 0) (effects (font (size 1.27 1.27)) (justify left bottom)))
+  (label "LOUT" (at 223.52 144.78 0) (effects (font (size 1.27 1.27)) (justify left bottom)))
+  (label "GATE" (at 242.57 144.78 0) (effects (font (size 1.27 1.27)) (justify left bottom)))
   (hierarchical_label "PWM_IN" (shape input) (at 162.56 154.94 0) (effects (font (size 1.27 1.27)) (justify right)))
   (hierarchical_label "ISENSE" (shape output) (at 283.21 165.1 0) (effects (font (size 1.27 1.27)) (justify left)))
