File: circuits/power_io.kicad_sch (KiCad schematic)
At the start: 55 parts, among them J5 24V DC IN, J6 CONN_RJ45, U11 AP2112K-3.3, U12 INA4180A1, U13 LM4040C50 5V, U14 AD7606BSTZ-4, U15 AP63205WU-7 5V BUCK, U16 AP63200WU-7 9.3V BUCK

Commit message: Checkpoint schematic warning hygiene
Parts:
- removed J6: CONN_RJ45, Connector_RJ:RJ45_Amphenol_RJHSE538X, symbol open_automation:CONN_RJ45
- added C65: 22uF 5V buck, Capacitor_SMD:C_0805_2012Metric_Pad1.18x1.45mm_HandSolder, symbol viv:C_V
- J6: renamed from C65; value 22uF 5V buck -> CONN_RJ45; footprint Capacitor_SMD:C_0805_2012Metric_Pad1.18x1.45mm_HandSolder -> Connector_RJ:RJ45_Amphenol_RJHSE538X; symbol viv:C_V -> open_automation:CONN_RJ45; LCSC C45783 -> C386757; Part Number CL21A226MAQNNNE -> R-RJ45R08P-C000
Connections:
- net BUCK_5V: now also C65.1; no longer J6.1
- net GND: now also J6.11, J6.4, J6.5, J6.7, J6.8, J6.9, C65.2; no longer J6.2
- net RJ45_LED_CONTACT: now also J6.12
- net RJ45_PWR_DETECT: now also J6.10
Changed lines of the file:
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@@
   (wire (pts (xy 82.55 143.51) (xy 105.41 143.51)) (stroke (width 0) (type default)))
   (wire (pts (xy 82.55 143.51) (xy 82.55 149.86)) (stroke (width 0) (type default)))
-  (wire (pts (xy 63.5 115.57) (xy 72.39 115.57)) (stroke (width 0) (type default)))
+  (wire (pts (xy 63.5 115.57) (xy 67.31 115.57)) (stroke (width 0) (type default)))
+  (wire (pts (xy 67.31 115.57) (xy 72.39 115.57)) (stroke (width 0) (type default)))
   (wire (pts (xy 72.39 115.57) (xy 72.39 116.84)) (stroke (width 0) (type default)))
-  (wire (pts (xy 63.5 134.62) (xy 72.39 134.62)) (stroke (width 0) (type default)))
+  (wire (pts (xy 67.31 115.57) (xy 67.31 110.49)) (stroke (width 0) (type default)))
+  (wire (pts (xy 63.5 134.62) (xy 67.31 134.62)) (stroke (width 0) (type default)))
+  (wire (pts (xy 67.31 134.62) (xy 72.39 134.62)) (stroke (width 0) (type default)))
   (wire (pts (xy 72.39 134.62) (xy 72.39 132.08)) (stroke (width 0) (type default)))
+  (wire (pts (xy 67.31 134.62) (xy 67.31 144.78)) (stroke (width 0) (type default)))
   (wire (pts (xy 55.88 115.57) (xy 55.88 106.68)) (stroke (width 0) (type default)))
   (wire (pts (xy 55.88 134.62) (xy 55.88 128.27)) (stroke (width 0) (type default)))
@@
   (wire (pts (xy 308.61 284.48) (xy 308.61 285.75)) (stroke (width 0) (type default)))
   (wire (pts (xy 308.61 285.75) (xy 285.75 285.75)) (stroke (width 0) (type default)))
+  (wire (pts (xy 285.75 285.75) (xy 275.59 285.75)) (stroke (width 0) (type default)))
   (wire (pts (xy 285.75 290.83) (xy 285.75 295.91)) (stroke (width 0) (type default)))
   (wire (pts (xy 317.5 289.56) (xy 308.61 289.56)) (stroke (width 0) (type default)))
   (wire (pts (xy 308.61 289.56) (xy 308.61 292.1)) (stroke (width 0) (type default)))
   (wire (pts (xy 308.61 292.1) (xy 274.32 292.1)) (stroke (width 0) (type default)))
+  (wire (pts (xy 274.32 292.1) (xy 264.16 292.1)) (stroke (width 0) (type default)))
   (wire (pts (xy 274.32 297.18) (xy 274.32 302.26)) (stroke (width 0) (type default)))
   (wire (pts (xy 317.5 294.64) (xy 308.61 294.64)) (stroke (width 0) (type default)))
   (wire (pts (xy 308.61 294.64) (xy 308.61 298.45)) (stroke (width 0) (type default)))
   (wire (pts (xy 308.61 298.45) (xy 261.62 298.45)) (stroke (width 0) (type default)))
+  (wire (pts (xy 261.62 298.45) (xy 251.46 298.45)) (stroke (width 0) (type default)))
   (wire (pts (xy 261.62 303.53) (xy 261.62 308.61)) (stroke (width 0) (type default)))
   (wire (pts (xy 317.5 299.72) (xy 308.61 299.72)) (stroke (width 0) (type default)))
@@
   (wire (pts (xy 308.61 299.72) (xy 308.61 304.8)) (stroke (width 0) (type default)))
   (wire (pts (xy 308.61 304.8) (xy 248.92 304.8)) (stroke (width 0) (type default)))
+  (wire (pts (xy 248.92 304.8) (xy 238.76 304.8)) (stroke (width 0) (type default)))
   (wire (pts (xy 248.92 309.88) (xy 248.92 314.96)) (stroke (width 0) (type default)))
   (wire (pts (xy 252.73 162.56) (xy 252.73 157.48)) (stroke (width 0) (type default)))
@@
   (junction (at 105.41 143.51) (diameter 0) (color 0 0 0 0))
   (junction (at 82.55 143.51) (diameter 0) (color 0 0 0 0))
+  (junction (at 67.31 115.57) (diameter 0) (color 0 0 0 0))
+  (junction (at 67.31 134.62) (diameter 0) (color 0 0 0 0))
   (junction (at 281.94 110.49) (diameter 0) (color 0 0 0 0))
   (junction (at 281.94 87.63) (diameter 0) (color 0 0 0 0))
@@
   (no_connect (at 337.82 101.6))
   (no_connect (at 368.3 274.32))
-  (label "RJ45_PWR_DETECT" (at 63.5 115.57 0) (effects (font (size 1.27 1.27)) (justify right bottom)))
-  (label "RJ45_LED_CONTACT" (at 63.5 134.62 0) (effects (font (size 1.27 1.27)) (justify right bottom)))
+  (label "RJ45_PWR_DETECT" (at 67.31 110.49 0) (effects (font (size 1.27 1.27)) (justify right bottom)))
+  (label "RJ45_LED_CONTACT" (at 67.31 144.78 0) (effects (font (size 1.27 1.27)) (justify right bottom)))
   (label "BUCK5_SW" (at 171.45 90.17 0) (effects (font (size 1.27 1.27)) (justify left bottom)))
   (label "BUCK5_BST" (at 171.45 95.25 0) (effects (font (size 1.27 1.27)) (justify left bottom)))
@@
   (hierarchical_label "ADC_MISO_A" (shape output) (at 378.46 276.86 0) (effects (font (size 1.27 1.27)) (justify left)))
   (hierarchical_label "ADC_MISO_B" (shape output) (at 378.46 279.4 0) (effects (font (size 1.27 1.27)) (justify left)))
-  (label "ADC_CREG1" (at 285.75 285.75 0) (effects (font (size 1.27 1.27)) (justify left bottom)))
-  (label "ADC_CREG2" (at 274.32 292.1 0) (effects (font (size 1.27 1.27)) (justify left bottom)))
-  (label "ADC_CREFIN" (at 261.62 298.45 0) (effects (font (size 1.27 1.27)) (justify left bottom)))
-  (label "ADC_REFCAP" (at 248.92 304.8 0) (effects (font (size 1.27 1.27)) (justify left bottom)))
+  (label "ADC_CREG1" (at 275.59 285.75 0) (effects (font (size 1.27 1.27)) (justify right bottom)))
+  (label "ADC_CREG2" (at 264.16 292.1 0) (effects (font (size 1.27 1.27)) (justify right bottom)))
+  (label "ADC_CREFIN" (at 251.46 298.45 0) (effects (font (size 1.27 1.27)) (justify right bottom)))
+  (label "ADC_REFCAP" (at 238.76 304.8 0) (effects (font (size 1.27 1.27)) (justify right bottom)))
   (label "MPD_BIAS" (at 162.56 177.8 0) (effects (font (size 1.27 1.27)) (justify right bottom)))
   (label "MPD_BIAS" (at 190.5 182.88 0) (effects (font (size 1.27 1.27)) (justify left bottom)))
@@
   (hierarchical_label "MPD_RAW1" (shape input) (at 307.34 157.48 0) (effects (font (size 1.27 1.27)) (justify right)))
   (label "MPD_BIAS" (at 340.36 157.48 0) (effects (font (size 1.27 1.27)) (justify left bottom)))
-  (label "MPD_RAW1" (at 231.14 167.64 0) (effects (font (size 1.27 1.27)) (justify right bottom)))
+  (hierarchical_label "MPD_RAW1" (shape input) (at 231.14 167.64 0) (effects (font (size 1.27 1.27)) (justify right)))
   (label "MPD_BIAS" (at 231.14 172.72 0) (effects (font (size 1.27 1.27)) (justify right bottom)))
   (label "MPD_AMP1" (at 276.86 170.18 0) (effects (font (size 1.27 1.27)) (justify left bottom)))
@@
   (hierarchical_label "MPD_RAW2" (shape input) (at 307.34 172.72 0) (effects (font (size 1.27 1.27)) (justify right)))
   (label "MPD_BIAS" (at 340.36 172.72 0) (effects (font (size 1.27 1.27)) (justify left bottom)))
-  (label "MPD_RAW2" (at 231.14 177.8 0) (effects (font (size 1.27 1.27)) (justify right bottom)))
+  (hierarchical_label "MPD_RAW2" (shape input) (at 231.14 177.8 0) (effects (font (size 1.27 1.27)) (justify right)))
   (label "MPD_BIAS" (at 231.14 182.88 0) (effects (font (size 1.27 1.27)) (justify right bottom)))
   (label "MPD_AMP2" (at 276.86 180.34 0) (effects (font (size 1.27 1.27)) (justify left bottom)))
@@
   (hierarchical_label "MPD_RAW3" (shape input) (at 307.34 187.96 0) (effects (font (size 1.27 1.27)) (justify right)))
   (label "MPD_BIAS" (at 340.36 187.96 0) (effects (font (size 1.27 1.27)) (justify left bottom)))
-  (label "MPD_RAW3" (at 231.14 187.96 0) (effects (font (size 1.27 1.27)) (justify right bottom)))
+  (hierarchical_label "MPD_RAW3" (shape input) (at 231.14 187.96 0) (effects (font (size 1.27 1.27)) (justify right)))
   (label "MPD_BIAS" (at 231.14 193.04 0) (effects (font (size 1.27 1.27)) (justify right bottom)))
   (label "MPD_AMP3" (at 276.86 190.5 0) (effects (font (size 1.27 1.27)) (justify left bottom)))
@@
   (hierarchical_label "MPD_RAW4" (shape input) (at 307.34 201.93 0) (effects (font (size 1.27 1.27)) (justify right)))
   (label "MPD_BIAS" (at 340.36 201.93 0) (effects (font (size 1.27 1.27)) (justify left bottom)))
-  (label "MPD_RAW4" (at 231.14 198.12 0) (effects (font (size 1.27 1.27)) (justify right bottom)))
+  (hierarchical_label "MPD_RAW4" (shape input) (at 231.14 198.12 0) (effects (font (size 1.27 1.27)) (justify right)))
   (label "MPD_BIAS" (at 231.14 203.2 0) (effects (font (size 1.27 1.27)) (justify right bottom)))
   (label "MPD_AMP4" (at 276.86 200.66 0) (effects (font (size 1.27 1.27)) (justify left bottom)))

Commit message: Prepare laser controller JLCPCB package
Parts:
- C70: LCSC C90264 -> C242011; Part Number RVT2A220M0810 -> 100CE22FS+P
- R41: LCSC C2099849 -> C103460; Part Number CRCW06032K49FKEAHP -> RTT032491FTP
- R42, R44, R46, R48: LCSC C114613 -> C103446; Part Number RC0603FR-07240RL -> RTT032400FTP
Changed lines of the file:
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@@
     (property "Footprint" "Capacitor_SMD:C_Elec_8x10.2" (at 144.78 85.09 0) (effects (font (size 1.0 1.0)) hide))
     (property "Datasheet" "" (at 144.78 85.09 0) (effects (font (size 1.0 1.0)) hide))
-    (property "Part Number" "RVT2A220M0810" (at 144.78 85.09 0) (effects (font (size 1.0 1.0)) hide))
-    (property "LCSC" "C90264" (at 144.78 85.09 0) (effects (font (size 1.0 1.0)) hide))
+    (property "Part Number" "100CE22FS+P" (at 144.78 85.09 0) (effects (font (size 1.0 1.0)) hide))
+    (property "LCSC" "C242011" (at 144.78 85.09 0) (effects (font (size 1.0 1.0)) hide))
     (pin "1")
     (pin "2")
@@
     (property "Footprint" "Resistor_SMD:R_0603_1608Metric_Pad0.98x0.95mm_HandSolder" (at 195.58 201.93 0) (effects (font (size 1.0 1.0)) hide))
     (property "Datasheet" "" (at 195.58 201.93 0) (effects (font (size 1.0 1.0)) hide))
-    (property "Part Number" "CRCW06032K49FKEAHP" (at 195.58 201.93 0) (effects (font (size 1.0 1.0)) hide))
-    (property "LCSC" "C2099849" (at 195.58 201.93 0) (effects (font (size 1.0 1.0)) hide))
+    (property "Part Number" "RTT032491FTP" (at 195.58 201.93 0) (effects (font (size 1.0 1.0)) hide))
+    (property "LCSC" "C103460" (at 195.58 201.93 0) (effects (font (size 1.0 1.0)) hide))
     (pin "1")
     (pin "2")
@@
     (property "Footprint" "Resistor_SMD:R_0603_1608Metric_Pad0.98x0.95mm_HandSolder" (at 325.12 157.48 0) (effects (font (size 1.0 1.0)) hide))
     (property "Datasheet" "" (at 325.12 157.48 0) (effects (font (size 1.0 1.0)) hide))
-    (property "Part Number" "RC0603FR-07240RL" (at 325.12 157.48 0) (effects (font (size 1.0 1.0)) hide))
-    (property "LCSC" "C114613" (at 325.12 157.48 0) (effects (font (size 1.0 1.0)) hide))
+    (property "Part Number" "RTT032400FTP" (at 325.12 157.48 0) (effects (font (size 1.0 1.0)) hide))
+    (property "LCSC" "C103446" (at 325.12 157.48 0) (effects (font (size 1.0 1.0)) hide))
     (pin "1")
     (pin "2")
@@
     (property "Footprint" "Resistor_SMD:R_0603_1608Metric_Pad0.98x0.95mm_HandSolder" (at 325.12 172.72 0) (effects (font (size 1.0 1.0)) hide))
     (property "Datasheet" "" (at 325.12 172.72 0) (effects (font (size 1.0 1.0)) hide))
-    (property "Part Number" "RC0603FR-07240RL" (at 325.12 172.72 0) (effects (font (size 1.0 1.0)) hide))
-    (property "LCSC" "C114613" (at 325.12 172.72 0) (effects (font (size 1.0 1.0)) hide))
+    (property "Part Number" "RTT032400FTP" (at 325.12 172.72 0) (effects (font (size 1.0 1.0)) hide))
+    (property "LCSC" "C103446" (at 325.12 172.72 0) (effects (font (size 1.0 1.0)) hide))
     (pin "1")
     (pin "2")
@@
     (property "Footprint" "Resistor_SMD:R_0603_1608Metric_Pad0.98x0.95mm_HandSolder" (at 325.12 187.96 0) (effects (font (size 1.0 1.0)) hide))
     (property "Datasheet" "" (at 325.12 187.96 0) (effects (font (size 1.0 1.0)) hide))
-    (property "Part Number" "RC0603FR-07240RL" (at 325.12 187.96 0) (effects (font (size 1.0 1.0)) hide))
-    (property "LCSC" "C114613" (at 325.12 187.96 0) (effects (font (size 1.0 1.0)) hide))
+    (property "Part Number" "RTT032400FTP" (at 325.12 187.96 0) (effects (font (size 1.0 1.0)) hide))
+    (property "LCSC" "C103446" (at 325.12 187.96 0) (effects (font (size 1.0 1.0)) hide))
     (pin "1")
     (pin "2")
@@
     (property "Footprint" "Resistor_SMD:R_0603_1608Metric_Pad0.98x0.95mm_HandSolder" (at 325.12 201.93 0) (effects (font (size 1.0 1.0)) hide))
     (property "Datasheet" "" (at 325.12 201.93 0) (effects (font (size 1.0 1.0)) hide))
-    (property "Part Number" "RC0603FR-07240RL" (at 325.12 201.93 0) (effects (font (size 1.0 1.0)) hide))
-    (property "LCSC" "C114613" (at 325.12 201.93 0) (effects (font (size 1.0 1.0)) hide))
-    (pin "1")
-    (pin "2")
+    (property "Part Number" "RTT032400FTP" (at 325.12 201.93 0) (effects (font (size 1.0 1.0)) hide))
+    (property "LCSC" "C103446" (at 325.12 201.93 0) (effects (font (size 1.0 1.0)) hide))
+    (pin "1")
+    (pin "2")

Commit message: Replace short-stock R41 assembly part
Parts:
- R41: LCSC C103460 -> C22908; Part Number RTT032491FTP -> 0603WAF2491T5E
Changed lines of the file:
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@@
     (property "Footprint" "Resistor_SMD:R_0603_1608Metric_Pad0.98x0.95mm_HandSolder" (at 195.58 201.93 0) (effects (font (size 1.0 1.0)) hide))
     (property "Datasheet" "" (at 195.58 201.93 0) (effects (font (size 1.0 1.0)) hide))
-    (property "Part Number" "RTT032491FTP" (at 195.58 201.93 0) (effects (font (size 1.0 1.0)) hide))
-    (property "LCSC" "C103460" (at 195.58 201.93 0) (effects (font (size 1.0 1.0)) hide))
+    (property "Part Number" "0603WAF2491T5E" (at 195.58 201.93 0) (effects (font (size 1.0 1.0)) hide))
+    (property "LCSC" "C22908" (at 195.58 201.93 0) (effects (font (size 1.0 1.0)) hide))
     (pin "1")
     (pin "2")

Commit message: Fix JLC assembly release for laser controller
Repair OPA380/Bourns orientation gates, substitute C70 with JLC C970665, and regenerate BOM/CPL/Gerber/JLC package artifacts.

Verified with run_laser_controller_review.py, check_jlcpcb_order_package.py, orientation/polarity PCB gate, and staged git diff whitespace check.
Parts:
- C70: LCSC C242011 -> C970665; Part Number 100CE22FS+P -> RVT2A220M0810 22UF 100V
Changed lines of the file:
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@@
     (property "Footprint" "Capacitor_SMD:C_Elec_8x10.2" (at 144.78 85.09 0) (effects (font (size 1.0 1.0)) hide))
     (property "Datasheet" "" (at 144.78 85.09 0) (effects (font (size 1.0 1.0)) hide))
-    (property "Part Number" "100CE22FS+P" (at 144.78 85.09 0) (effects (font (size 1.0 1.0)) hide))
-    (property "LCSC" "C242011" (at 144.78 85.09 0) (effects (font (size 1.0 1.0)) hide))
+    (property "Part Number" "RVT2A220M0810 22UF 100V" (at 144.78 85.09 0) (effects (font (size 1.0 1.0)) hide))
+    (property "LCSC" "C970665" (at 144.78 85.09 0) (effects (font (size 1.0 1.0)) hide))
     (pin "1")
     (pin "2")
